File: fa2_bit.kicad_sch (KiCad schematic)
At the start: 0 parts

Commit message: FA8 full sim, before FA1 layout
Changed lines of the file:
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@@
+	(wire
+		(pts
+			(xy 95.25 66.04) (xy 95.25 71.12)
+		)
+		(stroke
+			(width 0)
+			(type default)
+		)
+	)
 	(wire
 		(pts
@@
 	(wire
 		(pts
+			(xy 58.42 71.12) (xy 58.42 66.04)
+		)
+		(stroke
+			(width 0)
+			(type default)
+		)
+	)
+	(wire
+		(pts
+			(xy 102.87 90.17) (xy 102.87 93.98)
+		)
+		(stroke
+			(width 0)
+			(type default)
+		)
+	)
+	(wire
+		(pts
+			(xy 100.33 66.04) (xy 100.33 71.12)
+		)
+		(stroke
+			(width 0)
+			(type default)
+		)
+	)
+	(wire
+		(pts
 			(xy 101.6 120.65) (xy 104.14 120.65)
 		)
@@
 	(wire
 		(pts
+			(xy 97.79 90.17) (xy 97.79 93.98)
+		)
+		(stroke
+			(width 0)
+			(type default)
+		)
+	)
+	(wire
+		(pts
 			(xy 101.6 118.11) (xy 104.14 118.11)
 		)
@@
 		)
 	)
+	(wire
+		(pts
+			(xy 93.98 93.98) (xy 93.98 90.17)
+		)
+		(stroke
+			(width 0)
+			(type default)
+		)
+	)
 	(bus
 		(pts
@@
 		)
 	)
+	(wire
+		(pts
+			(xy 73.66 93.98) (xy 93.98 93.98)
+		)
+		(stroke
+			(width 0)
+			(type default)
+		)
+	)
 	(bus
 		(pts
@@
 			(width 0)
 			(type default)
+		)
+	)
+	(wire
+		(pts
+			(xy 58.42 66.04) (xy 73.66 66.04)
+		)
+		(stroke
+			(width 0)
+			(type default)
+		)
+	)
+	(wire
+		(pts
+			(xy 73.66 66.04) (xy 73.66 93.98)
+		)
+		(stroke
+			(width 0)
+			(type default)
+		)
+	)
+	(label "OUT_SUM1"
+		(at 95.25 66.04 90)
+		(effects
+			(font
+				(size 1.27 1.27)
+			)
+			(justify left bottom)
 		)
 	)
@@
 		)
 	)
+	(label "IN_B1"
+		(at 102.87 93.98 270)
+		(effects
+			(font
+				(size 1.27 1.27)
+			)
+			(justify right bottom)
+		)
+	)
 	(label "OUT_SUM0"
 		(at 104.14 118.11 0)
@@
 			)
 			(justify left bottom)
+		)
+	)
+	(label "IN_A1"
+		(at 97.79 93.98 270)
+		(effects
+			(font
+				(size 1.27 1.27)
+			)
+			(justify right bottom)
 		)
 	)
@@
 		)
 	)
+	(hierarchical_label "OUT_COUT"
+		(shape output)
+		(at 100.33 66.04 90)
+		(effects
+			(font
+				(size 1.27 1.27)
+			)
+			(justify left)
+		)
+	)

Commit message: FA 1-Bit PCB ok
Other:
- removed sheet fa2
