File: ICD24_FA.kicad_sch (KiCad schematic)
At the start: 0 parts

Commit message: full, no layout
Parts:
- added V1: 5, symbol Simulation_SPICE:VDC
Connections:
- new net 0: V1.2
- new net VDD: V1.1
Other:
- removed sheet and_gate
- removed sheet inverter
- removed sheet nand_gate
- removed sheet or_gate
- removed sheet xnor_gate
- removed sheet xor_gate
- added sheet board_interface (board_interface.kicad_sch)
- added sheet fa8 (fa8.kicad_sch)
- added sheet testbench_fa1 (testbench_fa1.kicad_sch)
- added sheet testbench_fa8 (testbench_fa8.kicad_sch)
- added sheet testbench_fa9 (testbench_fa8.kicad_sch)
- added sheet testbench_gates (testbench_gates.kicad_sch)

Commit message: FA 2-bit
Parts:
- renumbered V1 to V81
Other:
- removed sheet testbench_fa9
- added sheet fa2_bit (fa2_bit.kicad_sch)
- added sheet testbench_fa8_full (testbench_fa8_full.kicad_sch)

Commit message: FA8 full sim, before FA1 layout
Changed lines of the file:
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@@
 	)
 	(sheet
-		(at 127 25.4)
+		(at 130.81 25.4)
 		(size 21.59 13.97)
 		(exclude_from_sim no)
@@
 		)
 		(property "Sheetname" "testbench_fa8_full"
-			(at 127 24.6884 0)
+			(at 130.81 24.6884 0)
 			(effects
 				(font
@@
 		)
 		(property "Sheetfile" "testbench_fa8_full.kicad_sch"
-			(at 127 39.9546 0)
+			(at 130.81 39.9546 0)
 			(effects
 				(font
@@
 		(at 143.51 107.95)
 		(size 29.21 15.24)
-		(exclude_from_sim no)
+		(exclude_from_sim yes)
 		(in_bom yes)
 		(on_board yes)

Commit message: FA 1-Bit PCB ok
Other:
- sheet fa2_bit renamed fa1_bit
- sheet fa1_bit ports: added IN_A0, IN_B0, OUT_SUM0; removed IN_A[0..1], IN_B[0..1], OUT_SUM[0..1]
Changed lines of the file:
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@@
 	(paper "A4")
-	(junction
-		(at 143.51 119.38)
-		(diameter 0)
-		(color 0 0 0 0)
-	)
 	(junction
 		(at 193.04 41.91)
@@
 	(wire
 		(pts
+			(xy 138.43 119.38) (xy 143.51 119.38)
+		)
+		(stroke
+			(width 0)
+			(type default)
+		)
+	)
+	(wire
+		(pts
 			(xy 198.12 58.42) (xy 198.12 57.15)
 		)
@@
 		)
 	)
+	(wire
+		(pts
+			(xy 193.04 57.15) (xy 193.04 58.42)
+		)
+		(stroke
+			(width 0)
+			(type default)
+		)
+	)
 	(bus
 		(pts
+			(xy 138.43 87.63) (xy 144.78 87.63)
+		)
+		(stroke
+			(width 0)
+			(type default)
+		)
+	)
+	(wire
+		(pts
+			(xy 138.43 80.01) (xy 144.78 80.01)
+		)
+		(stroke
+			(width 0)
+			(type default)
+		)
+	)
+	(bus
+		(pts
+			(xy 138.43 83.82) (xy 144.78 83.82)
+		)
+		(stroke
+			(width 0)
+			(type default)
+		)
+	)
+	(wire
+		(pts
+			(xy 172.72 116.84) (xy 176.53 116.84)
+		)
+		(stroke
+			(width 0)
+			(type default)
+		)
+	)
+	(wire
+		(pts
+			(xy 193.04 54.61) (xy 193.04 57.15)
+		)
+		(stroke
+			(width 0)
+			(type default)
+		)
+	)
+	(wire
+		(pts
+			(xy 172.72 82.55) (xy 176.53 82.55)
+		)
+		(stroke
+			(width 0)
+			(type default)
+		)
+	)
+	(wire
+		(pts
+			(xy 193.04 40.64) (xy 193.04 41.91)
+		)
+		(stroke
+			(width 0)
+			(type default)
+		)
+	)
+	(wire
+		(pts
+			(xy 137.16 111.76) (xy 143.51 111.76)
+		)
+		(stroke
+			(width 0)
+			(type default)
+		)
+	)
+	(wire
+		(pts
+			(xy 172.72 111.76) (xy 176.53 111.76)
+		)
+		(stroke
+			(width 0)
+			(type default)
+		)
+	)
+	(wire
+		(pts
+			(xy 193.04 41.91) (xy 193.04 44.45)
+		)
+		(stroke
+			(width 0)
+			(type default)
+		)
+	)
+	(wire
+		(pts
+			(xy 198.12 57.15) (xy 193.04 57.15)
+		)
+		(stroke
+			(width 0)
+			(type default)
+		)
+	)
+	(wire
+		(pts
 			(xy 137.16 115.57) (xy 143.51 115.57)
 		)
@@
 	(wire
 		(pts
-			(xy 193.04 57.15) (xy 193.04 58.42)
-		)
-		(stroke
-			(width 0)
-			(type default)
-		)
-	)
-	(wire
-		(pts
-			(xy 138.43 119.38) (xy 143.51 119.38)
-		)
-		(stroke
-			(width 0)
-			(type default)
-		)
-	)
-	(bus
-		(pts
-			(xy 138.43 87.63) (xy 144.78 87.63)
-		)
-		(stroke
-			(width 0)
-			(type default)
-		)
-	)
-	(wire
-		(pts
-			(xy 138.43 80.01) (xy 144.78 80.01)
-		)
-		(stroke
-			(width 0)
-			(type default)
-		)
-	)
-	(bus
-		(pts
-			(xy 137.16 111.76) (xy 143.51 111.76)
-		)
-		(stroke
-			(width 0)
-			(type default)
-		)
-	)
-	(bus
-		(pts
-			(xy 138.43 83.82) (xy 144.78 83.82)
-		)
-		(stroke
-			(width 0)
-			(type default)
-		)
-	)
-	(wire
-		(pts
-			(xy 193.04 54.61) (xy 193.04 57.15)
-		)
-		(stroke
-			(width 0)
-			(type default)
-		)
-	)
-	(wire
-		(pts
-			(xy 172.72 82.55) (xy 176.53 82.55)
-		)
-		(stroke
-			(width 0)
-			(type default)
-		)
-	)
-	(wire
-		(pts
-			(xy 193.04 40.64) (xy 193.04 41.91)
-		)
-		(stroke
-			(width 0)
-			(type default)
-		)
-	)
-	(bus
-		(pts
-			(xy 172.72 116.84) (xy 176.53 116.84)
-		)
-		(stroke
-			(width 0)
-			(type default)
-		)
-	)
-	(wire
-		(pts
-			(xy 172.72 111.76) (xy 176.53 111.76)
-		)
-		(stroke
-			(width 0)
-			(type default)
-		)
-	)
-	(wire
-		(pts
-			(xy 193.04 41.91) (xy 193.04 44.45)
-		)
-		(stroke
-			(width 0)
-			(type default)
-		)
-	)
-	(wire
-		(pts
-			(xy 198.12 57.15) (xy 193.04 57.15)
-		)
-		(stroke
-			(width 0)
-			(type default)
-		)
-	)
-	(wire
-		(pts
 			(xy 198.12 58.42) (xy 217.17 58.42)
-		)
-		(stroke
-			(width 0)
-			(type default)
-		)
-	)
-	(wire
-		(pts
-			(xy 143.51 119.38) (xy 143.5288 119.38)
 		)
 		(stroke
@@
 		)
 	)
-	(global_label "OUT_SUM[0..1]"
+	(global_label "OUT_SUM0"
 		(shape output)
 		(at 176.53 116.84 0)
@@
 		)
 		(property "Intersheetrefs" "${INTERSHEET_REFS}"
-			(at 193.4248 116.84 0)
+			(at 189.3123 116.84 0)
 			(effects
 				(font
@@
 		)
 	)
-	(global_label "IN_B[0..1]"
+	(global_label "IN_B0"
 		(shape input)
 		(at 137.16 115.57 180)
@@
 		)
 		(property "Intersheetrefs" "${INTERSHEET_REFS}"
-			(at 124.6799 115.57 0)
+			(at 128.7924 115.57 0)
 			(effects
 				(font
@@
 		)
 	)
-	(global_label "IN_A[0..1]"
+	(global_label "IN_A0"
 		(shape input)
 		(at 137.16 111.76 180)
@@
 		)
 		(property "Intersheetrefs" "${INTERSHEET_REFS}"
-			(at 124.8613 111.76 0)
+			(at 128.9738 111.76 0)
 			(effects
 				(font
@@
 			(color 0 0 0 0.0000)
 		)
-		(property "Sheetname" "fa2_bit"
+		(property "Sheetname" "fa1_bit"
 			(at 143.51 107.2384 0)
 			(effects
@@
 			)
 		)
-		(pin "IN_A[0..1]" input
-			(at 143.51 111.76 180)
-			(effects
-				(font
-					(size 1.27 1.27)
-				)
-				(justify left)
-			)
-		)
-		(pin "IN_B[0..1]" input
-			(at 143.51 115.57 180)
-			(effects
-				(font
-					(size 1.27 1.27)
-				)
-				(justify left)
-			)
-		)
 		(pin "OUT_COUT" output
 			(at 172.72 111.76 0)
@@
 			)
 		)
-		(pin "OUT_SUM[0..1]" output
+		(pin "OUT_SUM0" output
 			(at 172.72 116.84 0)
 			(effects
@@
 			)
 		)
+		(pin "IN_B0" input
+			(at 143.51 115.57 180)
+			(effects
+				(font
+					(size 1.27 1.27)
+				)
+				(justify left)
+			)
+		)
+		(pin "IN_A0" input
+			(at 143.51 111.76 180)
+			(effects
+				(font
+					(size 1.27 1.27)
+				)
+				(justify left)
+			)
+		)

Commit message: BOM and Picture
Other:
- added sheet Extensive Equipments (untitled.kicad_sch)
Changed lines of the file:
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@@
+			)
+		)
+		(property "Equipment Link" ""
+			(at 193.04 49.53 0)
+			(effects
+				(font
+					(size 1.27 1.27)
+				)
+				(hide yes)
 			)
 		)
@@
 				)
 			)
+		)
+	)
+	(sheet
+		(at 91.44 107.95)
+		(size 30.48 17.78)
+		(exclude_from_sim yes)
+		(in_bom yes)
+		(on_board no)
+		(dnp no)
+		(fields_autoplaced yes)
+		(stroke
+			(width 0.1524)
+			(type solid)
+		)
+		(fill
+			(color 0 0 0 0.0000)
+		)
+		(property "Sheetname" "Extensive Equipments"
+			(at 91.44 107.2384 0)
+			(effects
+				(font
+					(size 1.27 1.27)
+				)
+				(justify left bottom)
+			)
+		)
+		(property "Sheetfile" "untitled.kicad_sch"
+			(at 91.44 126.3146 0)
+			(effects
+				(font
+					(size 1.27 1.27)
+				)
+				(justify left top)
+			)
+		)
+		(instances
+			(project "ICD24_FA"
+				(path "/b041be17-3693-4432-854e-c071e14fa049"
+					(page "173")
+				)
+			)
