File: and_gate.kicad_sch (KiCad schematic)
At the start: 7 parts, among them Q2 2N3904, Q3 2N3904, Q6 2N3904

Commit message: full, no layout
Parts:
- removed Q6: 2N3904, Package_TO_SOT_THT:TO-92_Inline, symbol Transistor_BJT:2N3904
- added Q1: 2N3904, Package_TO_SOT_THT:TO-92_Inline, symbol Transistor_BJT:2N3904
- renumbered R2 to R1, R3 to R2, R9 to R3
Connections:
- net GND: now also Q2.1 (E)
- net at R2.2: now also Q2.2 (B)
- net at R1.2: now also Q1.2 (B); no longer Q2.2 (B)
- net at Q3.2 (B), R3.2: now also Q1.3 (C); no longer Q2.3 (C)
- new net: Q1.1 (E), Q2.3 (C)

Commit message: FA 2-bit
Parts:
- renumbered Q3 to Q81, Q1 to Q82, Q2 to Q83, R3 to R81, R4 to R82, R1 to R83, R2 to R84

Commit message: FA8 full sim, before FA1 layout
Parts:
- Q81, Q82, Q83: footprint Package_TO_SOT_THT:TO-92_Inline -> MyLibrary:TO-92_Inline
Changed lines of the file:
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@@
 			)
 		)
-		(property "Footprint" "Package_TO_SOT_THT:TO-92_Inline"
+		(property "Footprint" "MyLibrary:TO-92_Inline"
 			(at 106.68 80.645 0)
 			(effects
@@
 			)
 		)
-		(property "Datasheet" "https://www.onsemi.com/pub/Collateral/2N3903-D.PDF"
+		(property "Datasheet" ""
 			(at 101.6 78.74 0)
 			(effects
@@
 			)
 		)
-		(property "Description" "0.2A Ic, 40V Vce, Small Signal NPN Transistor, TO-92"
+		(property "Description" ""
 			(at 101.6 78.74 0)
 			(effects
@@
 			)
 		)
-		(property "Footprint" "Package_TO_SOT_THT:TO-92_Inline"
+		(property "Footprint" "MyLibrary:TO-92_Inline"
 			(at 128.27 57.785 0)
 			(effects
@@
 			)
 		)
-		(property "Datasheet" "https://www.onsemi.com/pub/Collateral/2N3903-D.PDF"
+		(property "Datasheet" ""
 			(at 123.19 55.88 0)
 			(effects
@@
 			)
 		)
-		(property "Description" "0.2A Ic, 40V Vce, Small Signal NPN Transistor, TO-92"
+		(property "Description" ""
 			(at 123.19 55.88 0)
 			(effects
@@
 			)
 		)
-		(property "Footprint" "Package_TO_SOT_THT:TO-92_Inline"
+		(property "Footprint" "MyLibrary:TO-92_Inline"
 			(at 106.68 64.135 0)
 			(effects
@@
 			)
 		)
-		(property "Datasheet" "https://www.onsemi.com/pub/Collateral/2N3903-D.PDF"
+		(property "Datasheet" ""
 			(at 101.6 62.23 0)
 			(effects
@@
 			)
 		)
-		(property "Description" "0.2A Ic, 40V Vce, Small Signal NPN Transistor, TO-92"
+		(property "Description" ""
 			(at 101.6 62.23 0)
 			(effects

Commit message: BOM and Picture
Parts:
- Q81, Q82, Q83: Equipment Link (none) -> https://www.thegioiic.com/2n3904-transistor-npn-40v-0-2a-3-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
- R81, R83, R84: Equipment Link (none) -> https://www.thegioiic.com/dien-tro-220-kohm-1-4w-1-5-vong-m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
- R82: Equipment Link (none) -> https://www.thegioiic.com/dien-tro-47-kohm-1-2w-5-4-vong-mau
Changed lines of the file:
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@@
+			)
+		)
+		(property "Equipment Link" "https://www.thegioiic.com/2n3904-transistor-npn-40v-0-2a-3-chan-to-92"
+			(at 101.6 78.74 0)
+			(effects
+				(font
+					(size 1.27 1.27)
+				)
+				(hide yes)
 			)
 		)
@@
 			)
 		)
+		(property "Equipment Link" "https://www.thegioiic.com/dien-tro-220-kohm-1-4w-1-5-vong-mau"
+			(at 83.82 78.74 0)
+			(effects
+				(font
+					(size 1.27 1.27)
+				)
+				(hide yes)
+			)
+		)
 		(pin "2"
 		)
@@
 			)
 		)
+		(property "Equipment Link" "https://www.thegioiic.com/dien-tro-220-kohm-1-4w-1-5-vong-mau"
+			(at 104.14 41.91 0)
+			(effects
+				(font
+					(size 1.27 1.27)
+				)
+				(hide yes)
+			)
+		)
 		(pin "2"
 		)
@@
 			)
 		)
+		(property "Equipment Link" "https://www.thegioiic.com/dien-tro-220-kohm-1-4w-1-5-vong-mau"
+			(at 83.82 62.23 0)
+			(effects
+				(font
+					(size 1.27 1.27)
+				)
+				(hide yes)
+			)
+		)
 		(pin "2"
 		)
@@
 			)
 		)
+		(property "Equipment Link" "https://www.thegioiic.com/2n3904-transistor-npn-40v-0-2a-3-chan-to-92"
+			(at 123.19 55.88 0)
+			(effects
+				(font
+					(size 1.27 1.27)
+				)
+				(hide yes)
+			)
+		)
 		(pin "2"
 		)
@@
 			)
 		)
+		(property "Equipment Link" "https://www.thegioiic.com/2n3904-transistor-npn-40v-0-2a-3-chan-to-92"
+			(at 101.6 62.23 0)
+			(effects
+				(font
+					(size 1.27 1.27)
+				)
+				(hide yes)
+			)
+		)
 		(pin "2"
 		)
@@
 			(at 125.73 43.18 0)
 			(effects
+				(font
+					(size 1.27 1.27)
+				)
+				(hide yes)
+			)
+		)
+		(property "Equipment Link" "https://www.thegioiic.com/dien-tro-47-kohm-1-2w-5-4-vong-mau"
+			(at 125.73 43.18 0)
+			(effects
