File: board_interface.kicad_sch (KiCad schematic)
At the start: 70 parts, among them J1 Conn_01x02, SW1 SW_SPDT, SW10 SW_SPDT, SW11 SW_SPDT, SW12 SW_SPDT, SW13 SW_SPDT, SW14 SW_SPDT, SW15 SW_SPDT, SW16 SW_SPDT, SW17 SW_SPDT, SW2 SW_SPDT, SW3 SW_SPDT, SW4 SW_SPDT, SW5 SW_SPDT, SW6 SW_SPDT, SW7 SW_SPDT, SW8 SW_SPDT, SW9 SW_SPDT

Commit message: FA 2-bit
Parts:
- renumbered D14 to D100, D23 to D101, D7 to D102, D15 to D103, D24 to D104, D26 to D105, D25 to D106, D8 to D81, D16 to D82, D17 to D83, D1 to D84, D9 to D85, D18 to D86, D2 to D87, D10 to D88, D19 to D89, D3 to D90, D11 to D91, D20 to D92, D4 to D93, D12 to D94, D21 to D95, D5 to D96, D13 to D97, D22 to D98, D6 to D99, J1 to J81, R64 to R137, R72 to R138, R73 to R139, R57 to R140, R65 to R141, R74 to R142, R58 to R143, R66 to R144, R75 to R145, R59 to R146, R67 to R147, R76 to R148, R60 to R149, R68 to R150, R77 to R151, R61 to R152, R69 to R153, R78 to R154, R62 to R155, R70 to R156, R79 to R157, R63 to R158, R71 to R159, R80 to R160, R754 to R161, R81 to R162, SW1 to SW81, SW9 to SW82, SW2 to SW83, SW10 to SW84, SW3 to SW85, SW11 to SW86, SW4 to SW87, SW12 to SW88, SW5 to SW89, SW13 to SW90, SW6 to SW91, SW14 to SW92, SW7 to SW93, SW15 to SW94, SW8 to SW95, SW16 to SW96, SW17 to SW97

Commit message: FA 1-Bit PCB ok
Parts:
- D84, D85, D86, R140, R141, R142, SW83, SW84: now left out of the parts list
- J81: footprint Connector_PinHeader_2.54mm:PinHeader_1x02_P2.54mm_Vertical -> Connector_PinHeader_2.54mm:PinHeader_1x02_P2.54mm_Horizontal; symbol Connector_Generic:Conn_01x02 -> Connector_Generic:Conn_01x06
Connections:
- net CIN: now also J81.4 (Pin_4), J81.5 (Pin_5); no longer SW97.2 (B)
- net OUT_COUT: now also J81.6 (Pin_6)
- new net CIN_Port: J81.3 (Pin_3), SW97.2 (B)
Changed lines of the file:
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@@
 		)
 	)
+	(global_label "CIN_Port"
+		(shape input)
+		(at 27.94 140.97 180)
+		(fields_autoplaced yes)
+		(effects
+			(font
+				(size 1.27 1.27)
+			)
+			(justify right)
+		)
+		(property "Intersheetrefs" "${INTERSHEET_REFS}"
+			(at 16.851 140.97 0)
+			(effects
+				(font
+					(size 1.27 1.27)
+				)
+				(justify right)
+				(hide yes)
+			)
+		)
+	)
 	(global_label "VDD"
 		(shape input)
@@
 		)
 	)
+	(global_label "CIN"
+		(shape input)
+		(at 27.94 143.51 180)
+		(fields_autoplaced yes)
+		(effects
+			(font
+				(size 1.27 1.27)
+			)
+			(justify right)
+		)
+		(property "Intersheetrefs" "${INTERSHEET_REFS}"
+			(at 21.7495 143.51 0)
+			(effects
+				(font
+					(size 1.27 1.27)
+				)
+				(justify right)
+				(hide yes)
+			)
+		)
+	)
 	(global_label "GND"
 		(shape input)
@@
 		)
 	)
+	(global_label "OUT_COUT"
+		(shape output)
+		(at 27.94 148.59 180)
+		(fields_autoplaced yes)
+		(effects
+			(font
+				(size 1.27 1.27)
+			)
+			(justify right)
+		)
+		(property "Intersheetrefs" "${INTERSHEET_REFS}"
+			(at 15.46 148.59 0)
+			(effects
+				(font
+					(size 1.27 1.27)
+				)
+				(justify right)
+				(hide yes)
+			)
+		)
+	)
 	(global_label "GND"
 		(shape input)
@@
 		)
 	)
+	(global_label "CIN"
+		(shape input)
+		(at 27.94 146.05 180)
+		(fields_autoplaced yes)
+		(effects
+			(font
+				(size 1.27 1.27)
+			)
+			(justify right)
+		)
+		(property "Intersheetrefs" "${INTERSHEET_REFS}"
+			(at 21.7495 146.05 0)
+			(effects
+				(font
+					(size 1.27 1.27)
+				)
+				(justify right)
+				(hide yes)
+			)
+		)
+	)
 	(global_label "VDD"
 		(shape input)
@@
 	(global_label "VDD"
 		(shape input)
-		(at 27.94 140.97 180)
+		(at 27.94 135.89 180)
 		(fields_autoplaced yes)
 		(effects
@@
 		)
 		(property "Intersheetrefs" "${INTERSHEET_REFS}"
-			(at 21.3262 140.97 0)
+			(at 21.3262 135.89 0)
 			(effects
 				(font
@@
 		)
 	)
-	(global_label "CIN"
+	(global_label "CIN_Port"
 		(shape input)
 		(at 91.44 146.05 180)
@@
 		)
 		(property "Intersheetrefs" "${INTERSHEET_REFS}"
-			(at 85.2495 146.05 0)
+			(at 80.351 146.05 0)
 			(effects
 				(font
@@
 	(global_label "GND"
 		(shape input)
-		(at 27.94 143.51 180)
+		(at 27.94 138.43 180)
 		(fields_autoplaced yes)
 		(effects
@@
 		)
 		(property "Intersheetrefs" "${INTERSHEET_REFS}"
-			(at 21.0843 143.51 0)
+			(at 21.0843 138.43 0)
 			(effects
 				(font
@@
 		(unit 1)
 		(exclude_from_sim no)
-		(in_bom yes)
-		(on_board yes)
+		(in_bom no)
+		(on_board no)
 		(dnp no)
 		(fields_autoplaced yes)
@@
 		(unit 1)
 		(exclude_from_sim no)
-		(in_bom yes)
-		(on_board yes)
+		(in_bom no)
+		(on_board no)
 		(dnp no)
 		(fields_autoplaced yes)
@@
 		(unit 1)
 		(exclude_from_sim no)
-		(in_bom yes)
-		(on_board yes)
+		(in_bom no)
+		(on_board no)
 		(dnp no)
 		(property "Reference" "D85"
@@
 		(unit 1)
 		(exclude_from_sim no)
-		(in_bom yes)
-		(on_board yes)
+		(in_bom no)
+		(on_board no)
 		(dnp no)
 		(property "Reference" "D84"
@@
 		(unit 1)
 		(exclude_from_sim no)
-		(in_bom yes)
-		(on_board yes)
+		(in_bom no)
+		(on_board no)
 		(dnp no)
 		(fields_autoplaced yes)
@@
 	)
 	(symbol
-		(lib_id "Connector_Generic:Conn_01x02")
+		(lib_id "Connector_Generic:Conn_01x06")
 		(at 33.02 140.97 0)
 		(unit 1)
@@
 			)
 		)
-		(property "Footprint" "Connector_PinHeader_2.54mm:PinHeader_1x02_P2.54mm_Vertical"
+		(property "Footprint" "Connector_PinHeader_2.54mm:PinHeader_1x02_P2.54mm_Horizontal"
 			(at 33.02 140.97 0)
 			(effects
@@
 			)
 		)
-		(property "Description" "Generic connector, single row, 01x02, script generated (kicad-library-utils/schlib/autogen/connector/)"
+		(property "Description" "Generic connector, single row, 01x06, script generated (kicad-library-utils/schlib/autogen/connector/)"
 			(at 33.02 140.97 0)
 			(effects
@@
 		(pin "2"
 		)
+		(pin "3"
+		)
+		(pin "4"
+		)
+		(pin "5"
+		)
+		(pin "6"
+		)
 		(instances
 			(project ""
@@
 		(unit 1)
 		(exclude_from_sim no)
-		(in_bom yes)
-		(on_board yes)
+		(in_bom no)
+		(on_board no)
 		(dnp no)
 		(fields_autoplaced yes)
@@
 		(unit 1)
 		(exclude_from_sim no)
-		(in_bom yes)
-		(on_board yes)
+		(in_bom no)
+		(on_board no)
 		(dnp no)
 		(fields_autoplaced yes)
@@
 		(unit 1)
 		(exclude_from_sim no)
-		(in_bom yes)
-		(on_board yes)
+		(in_bom no)
+		(on_board no)
 		(dnp no)
 		(fields_autoplaced yes)

Commit message: FA 1-bit PCB Ok
Parts:
- J81: value Conn_01x02 -> Conn_01x08; footprint Connector_PinHeader_2.54mm:PinHeader_1x02_P2.54mm_Horizontal -> Connector_PinHeader_2.54mm:PinHeader_1x08_P2.54mm_Horizontal; symbol Connector_Generic:Conn_01x06 -> Connector_Generic:Conn_01x08
Connections:
- net CIN: now also J81.6 (Pin_6), J81.7 (Pin_7); no longer J81.4 (Pin_4), J81.5 (Pin_5)
- net CIN_Port: now also J81.5 (Pin_5); no longer J81.3 (Pin_3)
- net GND: now also J81.3 (Pin_3), J81.4 (Pin_4); no longer J81.2 (Pin_2)
- net OUT_COUT: now also J81.8 (Pin_8); no longer J81.6 (Pin_6)
- net VDD: now also J81.2 (Pin_2)
Changed lines of the file:
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@@
 	(global_label "CIN_Port"
 		(shape input)
-		(at 27.94 140.97 180)
+		(at 27.94 143.51 180)
 		(fields_autoplaced yes)
 		(effects
@@
 		)
 		(property "Intersheetrefs" "${INTERSHEET_REFS}"
-			(at 16.851 140.97 0)
+			(at 16.851 143.51 0)
 			(effects
 				(font
@@
 	(global_label "CIN"
 		(shape input)
-		(at 27.94 143.51 180)
+		(at 27.94 146.05 180)
 		(fields_autoplaced yes)
 		(effects
@@
 		)
 		(property "Intersheetrefs" "${INTERSHEET_REFS}"
-			(at 21.7495 143.51 0)
+			(at 21.7495 146.05 0)
 			(effects
 				(font
@@
 	(global_label "OUT_COUT"
 		(shape output)
-		(at 27.94 148.59 180)
+		(at 27.94 151.13 180)
 		(fields_autoplaced yes)
 		(effects
@@
 		)
 		(property "Intersheetrefs" "${INTERSHEET_REFS}"
-			(at 15.46 148.59 0)
+			(at 15.46 151.13 0)
 			(effects
 				(font
@@
 	(global_label "CIN"
 		(shape input)
-		(at 27.94 146.05 180)
+		(at 27.94 148.59 180)
 		(fields_autoplaced yes)
 		(effects
@@
 		)
 		(property "Intersheetrefs" "${INTERSHEET_REFS}"
-			(at 21.7495 146.05 0)
+			(at 21.7495 148.59 0)
 			(effects
 				(font
@@
 		)
 	)
+	(global_label "GND"
+		(shape input)
+		(at 27.94 140.97 180)
+		(fields_autoplaced yes)
+		(effects
+			(font
+				(size 1.27 1.27)
+			)
+			(justify right)
+		)
+		(property "Intersheetrefs" "${INTERSHEET_REFS}"
+			(at 21.0843 140.97 0)
+			(effects
+				(font
+					(size 1.27 1.27)
+				)
+				(justify right)
+				(hide yes)
+			)
+		)
+	)
 	(global_label "VDD"
 		(shape input)
@@
 	(global_label "VDD"
 		(shape input)
-		(at 27.94 135.89 180)
+		(at 27.94 133.35 180)
 		(fields_autoplaced yes)
 		(effects
@@
 		)
 		(property "Intersheetrefs" "${INTERSHEET_REFS}"
-			(at 21.3262 135.89 0)
+			(at 21.3262 133.35 0)
 			(effects
 				(font
@@
 		)
 	)
+	(global_label "VDD"
+		(shape input)
+		(at 27.94 135.89 180)
+		(fields_autoplaced yes)
+		(effects
+			(font
+				(size 1.27 1.27)
+			)
+			(justify right)
+		)
+		(property "Intersheetrefs" "${INTERSHEET_REFS}"
+			(at 21.3262 135.89 0)
+			(effects
+				(font
+					(size 1.27 1.27)
+				)
+				(justify right)
+				(hide yes)
+			)
+		)
+	)
 	(global_label "GND"
 		(shape input)
@@
 	)
 	(symbol
-		(lib_id "Connector_Generic:Conn_01x06")
+		(lib_id "Connector_Generic:Conn_01x08")
 		(at 33.02 140.97 0)
 		(unit 1)
@@
 			)
 		)
-		(property "Value" "Conn_01x02"
+		(property "Value" "Conn_01x08"
 			(at 35.56 143.5099 0)
 			(effects
@@
 			)
 		)
-		(property "Footprint" "Connector_PinHeader_2.54mm:PinHeader_1x02_P2.54mm_Horizontal"
+		(property "Footprint" "Connector_PinHeader_2.54mm:PinHeader_1x08_P2.54mm_Horizontal"
 			(at 33.02 140.97 0)
 			(effects
@@
 			)
 		)
-		(property "Description" "Generic connector, single row, 01x06, script generated (kicad-library-utils/schlib/autogen/connector/)"
+		(property "Description" "Generic connector, single row, 01x08, script generated (kicad-library-utils/schlib/autogen/connector/)"
 			(at 33.02 140.97 0)
 			(effects
@@
 		(pin "6"
 		)
+		(pin "7"
+		)
+		(pin "8"
+		)
 		(instances

Commit message: BOM and Picture
Parts:
- D100, D101, D102, D103, D104, D105, D106, D81, D82, D83, D87, D88, D89, D90, D91, D92, D93, D94, D95, D96, D97, D98, D99: Equipment Link (none) -> https://nshopvn.com/product/led-duc-5mm-xanh-la-xanh-duong-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
- J81: Equipment Link (none) -> https://www.thegioiic.com/hang-rao-duc-don-2-54mm-40-chan-c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
- R137, R138, R139, R143, R144, R145, R146, R147, R148, R149, R150, R151, R152, R153, R154, R155, R156, R157, R158, R159, R160, R161, R162: Equipment Link (none) -> https://www.thegioiic.com/dien-tro-47-kohm-1-2w-5-4-vong-mau
- SW81, SW82, SW85, SW86, SW87, SW88, SW89, SW90, SW91, SW92, SW93, SW94, SW95, SW96, SW97: Equipment Link (none) -> https://www.thegioiic.com/ss-12d07vg4-cong-tac-truot-5-chan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
