File: inverter.kicad_sch (KiCad schematic)
At the start: 3 parts, among them Q4 2N3904

Commit message: full, no layout
Parts:
- renumbered R7 to R6
Changed lines of the file:
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@@
+			)
+		)
+		(property "Sim.Library" "2N3904_model.txt"
+			(at 147.32 81.28 0)
+			(effects
+				(font
+					(size 1.27 1.27)
+				)
+				(hide yes)
+			)
+		)
+		(property "Sim.Name" "2N3904"
+			(at 147.32 81.28 0)
+			(effects
+				(font
+					(size 1.27 1.27)
+				)
+				(hide yes)
+			)
+		)
+		(property "Sim.Device" "NPN"
+			(at 147.32 81.28 0)
+			(effects
+				(font
+					(size 1.27 1.27)
+				)
+				(hide yes)
+			)
+		)
+		(property "Sim.Type" "GUMMELPOON"
+			(at 147.32 81.28 0)
+			(effects
+				(font
+					(size 1.27 1.27)
+				)
+				(hide yes)
+			)
+		)
+		(property "Sim.Pins" "1=E 2=B 3=C"
+			(at 147.32 81.28 0)
+			(effects
+				(font
+					(size 1.27 1.27)
+				)
+				(hide yes)
 			)
 		)
@@
 		(instances
 			(project "ICD24_FA"
-				(path "/b041be17-3693-4432-854e-c071e14fa049/b7c2df59-ac61-486a-9460-5086e01633a1"
+				(path "/b041be17-3693-4432-854e-c071e14fa049/bf61237c-4d83-41f1-a6ca-83160467bc81/ccc6d5ad-8a58-4a59-ae4f-3b0ed0cb8f96"
 					(reference "Q4")
 					(unit 1)
@@
 		(instances
 			(project "ICD24_FA"
-				(path "/b041be17-3693-4432-854e-c071e14fa049/b7c2df59-ac61-486a-9460-5086e01633a1"
+				(path "/b041be17-3693-4432-854e-c071e14fa049/bf61237c-4d83-41f1-a6ca-83160467bc81/ccc6d5ad-8a58-4a59-ae4f-3b0ed0cb8f96"
 					(reference "R5")
 					(unit 1)
@@
 		(dnp no)
 		(fields_autoplaced yes)
-		(property "Reference" "R7"
+		(property "Reference" "R6"
 			(at 152.4 59.6899 0)
 			(effects
@@
 		(instances
 			(project "ICD24_FA"
-				(path "/b041be17-3693-4432-854e-c071e14fa049/b7c2df59-ac61-486a-9460-5086e01633a1"
-					(reference "R7")
+				(path "/b041be17-3693-4432-854e-c071e14fa049/bf61237c-4d83-41f1-a6ca-83160467bc81/ccc6d5ad-8a58-4a59-ae4f-3b0ed0cb8f96"
+					(reference "R6")
 					(unit 1)
 				)

Commit message: FA 2-bit
Parts:
- renumbered Q4 to Q84, R6 to R85, R5 to R86
Changed lines of the file:
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@@
 		(dnp no)
 		(fields_autoplaced yes)
-		(property "Reference" "Q4"
+		(property "Reference" "Q84"
 			(at 152.4 80.0099 0)
 			(effects
@@
 			(project "ICD24_FA"
 				(path "/b041be17-3693-4432-854e-c071e14fa049/bf61237c-4d83-41f1-a6ca-83160467bc81/ccc6d5ad-8a58-4a59-ae4f-3b0ed0cb8f96"
-					(reference "Q4")
+					(reference "Q84")
 					(unit 1)
 				)
@@
 		(dnp no)
 		(fields_autoplaced yes)
-		(property "Reference" "R5"
+		(property "Reference" "R86"
 			(at 128.2699 78.74 0)
 			(effects
@@
 			(project "ICD24_FA"
 				(path "/b041be17-3693-4432-854e-c071e14fa049/bf61237c-4d83-41f1-a6ca-83160467bc81/ccc6d5ad-8a58-4a59-ae4f-3b0ed0cb8f96"
-					(reference "R5")
+					(reference "R86")
 					(unit 1)
 				)
@@
 		(dnp no)
 		(fields_autoplaced yes)
-		(property "Reference" "R6"
+		(property "Reference" "R85"
 			(at 152.4 59.6899 0)
 			(effects
@@
 			(project "ICD24_FA"
 				(path "/b041be17-3693-4432-854e-c071e14fa049/bf61237c-4d83-41f1-a6ca-83160467bc81/ccc6d5ad-8a58-4a59-ae4f-3b0ed0cb8f96"
-					(reference "R6")
+					(reference "R85")
 					(unit 1)
 				)
