File: nand_gate.kicad_sch (KiCad schematic)
At the start: 5 parts, among them Q13 2N3904, Q14 2N3904

Commit message: full, no layout
Parts:
- removed Q13, Q14: 2N3904, Package_TO_SOT_THT:TO-92_Inline, symbol Transistor_BJT:2N3904
- added Q5, Q6: 2N3904, Package_TO_SOT_THT:TO-92_Inline, symbol Transistor_BJT:2N3904
- renumbered R19 to R7, R20 to R8, R21 to R9
Connections:
- net GND: now also Q6.1 (E)
- net OUT: now also Q5.3 (C)
- net at R7.2: now also Q5.2 (B)
- net at R8.2: now also Q6.2 (B)
- new net: Q5.1 (E), Q6.3 (C)

Commit message: FA 2-bit
Parts:
- renumbered Q5 to Q85, Q6 to Q86, R9 to R87, R7 to R88, R8 to R89
Changed lines of the file:
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@@
 		(dnp no)
 		(fields_autoplaced yes)
-		(property "Reference" "Q6"
+		(property "Reference" "Q86"
 			(at 128.27 97.7899 0)
 			(effects
@@
 			(project "ICD24_FA"
 				(path "/b041be17-3693-4432-854e-c071e14fa049/bf61237c-4d83-41f1-a6ca-83160467bc81/eadfb294-1476-429b-adc0-6437a7fea880"
-					(reference "Q6")
+					(reference "Q86")
 					(unit 1)
 				)
@@
 		(dnp no)
 		(fields_autoplaced yes)
-		(property "Reference" "R9"
+		(property "Reference" "R87"
 			(at 128.27 67.3099 0)
 			(effects
@@
 			(project "ICD24_FA"
 				(path "/b041be17-3693-4432-854e-c071e14fa049/bf61237c-4d83-41f1-a6ca-83160467bc81/eadfb294-1476-429b-adc0-6437a7fea880"
-					(reference "R9")
+					(reference "R87")
 					(unit 1)
 				)
@@
 		(dnp no)
 		(fields_autoplaced yes)
-		(property "Reference" "R7"
+		(property "Reference" "R88"
 			(at 104.1399 80.01 0)
 			(effects
@@
 			(project "ICD24_FA"
 				(path "/b041be17-3693-4432-854e-c071e14fa049/bf61237c-4d83-41f1-a6ca-83160467bc81/eadfb294-1476-429b-adc0-6437a7fea880"
-					(reference "R7")
+					(reference "R88")
 					(unit 1)
 				)
@@
 		(dnp no)
 		(fields_autoplaced yes)
-		(property "Reference" "R8"
+		(property "Reference" "R89"
 			(at 104.1399 96.52 0)
 			(effects
@@
 			(project "ICD24_FA"
 				(path "/b041be17-3693-4432-854e-c071e14fa049/bf61237c-4d83-41f1-a6ca-83160467bc81/eadfb294-1476-429b-adc0-6437a7fea880"
-					(reference "R8")
+					(reference "R89")
 					(unit 1)
 				)
@@
 		(dnp no)
 		(fields_autoplaced yes)
-		(property "Reference" "Q5"
+		(property "Reference" "Q85"
 			(at 128.27 81.2799 0)
 			(effects
@@
 			(project "ICD24_FA"
 				(path "/b041be17-3693-4432-854e-c071e14fa049/bf61237c-4d83-41f1-a6ca-83160467bc81/eadfb294-1476-429b-adc0-6437a7fea880"
-					(reference "Q5")
+					(reference "Q85")
 					(unit 1)
 				)
