File: or_gate.kicad_sch (KiCad schematic)
At the start: 7 parts, among them Q1 2N3904, Q5 2N3904, Q7 2N3904

Commit message: full, no layout
Parts:
- removed Q1, Q5: 2N3904, Package_TO_SOT_THT:TO-92_Inline, symbol Transistor_BJT:2N3904
- added Q8, Q9: 2N3904, Package_TO_SOT_THT:TO-92_Inline, symbol Transistor_BJT:2N3904
- renumbered R6 to R10, R1 to R11, R8 to R12, R10 to R13
Connections:
- net GND: now also Q8.1 (E), Q9.1 (E)
- net OUT: now also Q9.3 (C); no longer Q7.3 (C)
- net at R12.2: now also Q7.3 (C), Q8.3 (C), Q9.2 (B)
- net at R11.2: now also Q8.2 (B)
- net at R10.2: now also Q7.2 (B)

Commit message: FA 2-bit
Parts:
- renumbered Q9 to Q87, Q8 to Q88, Q7 to Q89, R12 to R90, R13 to R91, R11 to R92, R10 to R93

Commit message: FA8 full sim, before FA1 layout
Parts:
- Q87, Q88, Q89: footprint Package_TO_SOT_THT:TO-92_Inline -> MyLibrary:TO-92_Inline
Changed lines of the file:
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@@
 			)
 		)
-		(property "Footprint" "Package_TO_SOT_THT:TO-92_Inline"
+		(property "Footprint" "MyLibrary:TO-92_Inline"
 			(at 139.7 64.135 0)
 			(effects
@@
 			)
 		)
-		(property "Datasheet" "https://www.onsemi.com/pub/Collateral/2N3903-D.PDF"
+		(property "Datasheet" ""
 			(at 134.62 62.23 0)
 			(effects
@@
 			)
 		)
-		(property "Description" "0.2A Ic, 40V Vce, Small Signal NPN Transistor, TO-92"
+		(property "Description" ""
 			(at 134.62 62.23 0)
 			(effects
@@
 			)
 		)
-		(property "Footprint" "Package_TO_SOT_THT:TO-92_Inline"
+		(property "Footprint" "MyLibrary:TO-92_Inline"
 			(at 130.81 75.565 0)
 			(effects
@@
 			)
 		)
-		(property "Datasheet" "https://www.onsemi.com/pub/Collateral/2N3903-D.PDF"
+		(property "Datasheet" ""
 			(at 125.73 73.66 0)
 			(effects
@@
 			)
 		)
-		(property "Description" "0.2A Ic, 40V Vce, Small Signal NPN Transistor, TO-92"
+		(property "Description" ""
 			(at 125.73 73.66 0)
 			(effects
@@
 			)
 		)
-		(property "Footprint" "Package_TO_SOT_THT:TO-92_Inline"
+		(property "Footprint" "MyLibrary:TO-92_Inline"
 			(at 161.29 57.785 0)
 			(effects
@@
 			)
 		)
-		(property "Datasheet" "https://www.onsemi.com/pub/Collateral/2N3903-D.PDF"
+		(property "Datasheet" ""
 			(at 156.21 55.88 0)
 			(effects
@@
 			)
 		)
-		(property "Description" "0.2A Ic, 40V Vce, Small Signal NPN Transistor, TO-92"
+		(property "Description" ""
 			(at 156.21 55.88 0)
 			(effects

Commit message: BOM and Picture
Parts:
- Q87, Q88, Q89: Equipment Link (none) -> https://www.thegioiic.com/2n3904-transistor-npn-40v-0-2a-3-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
- R90, R92, R93: Equipment Link (none) -> https://www.thegioiic.com/dien-tro-220-kohm-1-4w-1-5-vong-m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
- R91: Equipment Link (none) -> https://www.thegioiic.com/dien-tro-47-kohm-1-2w-5-4-vong-mau
Changed lines of the file:
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@@
+			)
+		)
+		(property "Equipment Link" "https://www.thegioiic.com/2n3904-transistor-npn-40v-0-2a-3-chan-to-92"
+			(at 134.62 62.23 0)
+			(effects
+				(font
+					(size 1.27 1.27)
+				)
+				(hide yes)
 			)
 		)
@@
 			)
 		)
+		(property "Equipment Link" "https://www.thegioiic.com/dien-tro-220-kohm-1-4w-1-5-vong-mau"
+			(at 137.16 41.91 0)
+			(effects
+				(font
+					(size 1.27 1.27)
+				)
+				(hide yes)
+			)
+		)
 		(pin "2"
 		)
@@
 			)
 		)
+		(property "Equipment Link" "https://www.thegioiic.com/2n3904-transistor-npn-40v-0-2a-3-chan-to-92"
+			(at 125.73 73.66 0)
+			(effects
+				(font
+					(size 1.27 1.27)
+				)
+				(hide yes)
+			)
+		)
 		(pin "2"
 		)
@@
 			)
 		)
+		(property "Equipment Link" "https://www.thegioiic.com/2n3904-transistor-npn-40v-0-2a-3-chan-to-92"
+			(at 156.21 55.88 0)
+			(effects
+				(font
+					(size 1.27 1.27)
+				)
+				(hide yes)
+			)
+		)
 		(pin "2"
 		)
@@
 			)
 		)
+		(property "Equipment Link" "https://www.thegioiic.com/dien-tro-220-kohm-1-4w-1-5-vong-mau"
+			(at 116.84 62.23 0)
+			(effects
+				(font
+					(size 1.27 1.27)
+				)
+				(hide yes)
+			)
+		)
 		(pin "2"
 		)
@@
 			)
 		)
+		(property "Equipment Link" "https://www.thegioiic.com/dien-tro-47-kohm-1-2w-5-4-vong-mau"
+			(at 158.75 43.18 0)
+			(effects
+				(font
+					(size 1.27 1.27)
+				)
+				(hide yes)
+			)
+		)
 		(pin "2"
 		)
@@
 			(at 114.3 73.66 0)
 			(effects
+				(font
+					(size 1.27 1.27)
+				)
+				(hide yes)
+			)
+		)
+		(property "Equipment Link" "https://www.thegioiic.com/dien-tro-220-kohm-1-4w-1-5-vong-mau"
+			(at 114.3 73.66 0)
+			(effects
