File: testbench_fa1.kicad_sch (KiCad schematic)
At the start: 3 parts

Commit message: FA 2-bit
Parts:
- renumbered V4 to V84, V5 to V85, V6 to V86
Changed lines of the file:
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@@
 		(dnp no)
 		(fields_autoplaced yes)
-		(property "Reference" "V4"
+		(property "Reference" "V84"
 			(at 38.1 70.9901 0)
 			(effects
@@
 			(project "ICD24_FA"
 				(path "/b041be17-3693-4432-854e-c071e14fa049/ca11677b-10e0-4873-9630-591117a9d374"
-					(reference "V4")
+					(reference "V84")
 					(unit 1)
 				)
@@
 		(dnp no)
 		(fields_autoplaced yes)
-		(property "Reference" "#PWR05"
+		(property "Reference" "#PWR085"
 			(at 34.29 87.63 0)
 			(effects
@@
 			(project "ICD24_FA"
 				(path "/b041be17-3693-4432-854e-c071e14fa049/ca11677b-10e0-4873-9630-591117a9d374"
-					(reference "#PWR05")
+					(reference "#PWR085")
 					(unit 1)
 				)
@@
 		(dnp no)
 		(fields_autoplaced yes)
-		(property "Reference" "#PWR07"
+		(property "Reference" "#PWR087"
 			(at 34.29 139.7 0)
 			(effects
@@
 			(project "ICD24_FA"
 				(path "/b041be17-3693-4432-854e-c071e14fa049/ca11677b-10e0-4873-9630-591117a9d374"
-					(reference "#PWR07")
+					(reference "#PWR087")
 					(unit 1)
 				)
@@
 		(dnp no)
 		(fields_autoplaced yes)
-		(property "Reference" "#PWR06"
+		(property "Reference" "#PWR086"
 			(at 34.29 111.76 0)
 			(effects
@@
 			(project "ICD24_FA"
 				(path "/b041be17-3693-4432-854e-c071e14fa049/ca11677b-10e0-4873-9630-591117a9d374"
-					(reference "#PWR06")
+					(reference "#PWR086")
 					(unit 1)
 				)
@@
 		(dnp no)
 		(fields_autoplaced yes)
-		(property "Reference" "V5"
+		(property "Reference" "V85"
 			(at 38.1 96.3901 0)
 			(effects
@@
 			(project "ICD24_FA"
 				(path "/b041be17-3693-4432-854e-c071e14fa049/ca11677b-10e0-4873-9630-591117a9d374"
-					(reference "V5")
+					(reference "V85")
 					(unit 1)
 				)
@@
 		(dnp no)
 		(fields_autoplaced yes)
-		(property "Reference" "V6"
+		(property "Reference" "V86"
 			(at 38.1 124.3301 0)
 			(effects
@@
 			(project "ICD24_FA"
 				(path "/b041be17-3693-4432-854e-c071e14fa049/ca11677b-10e0-4873-9630-591117a9d374"
-					(reference "V6")
-					(unit 1)
-				)
+					(reference "V86")
+					(unit 1)
+				)
