File: testbench_fa8.kicad_sch (KiCad schematic)
At the start: 1 part

Commit message: FA 2-bit
Parts:
- renumbered V7 to V87
Changed lines of the file:
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@@
 		(dnp no)
 		(fields_autoplaced yes)
-		(property "Reference" "V7"
+		(property "Reference" "V87"
 			(at 46.99 74.8001 0)
 			(effects
@@
 			(project ""
 				(path "/b041be17-3693-4432-854e-c071e14fa049/79b0d0a7-c4a7-4cc5-bd2e-f49e97388b8b"
-					(reference "V7")
-					(unit 1)
-				)
-				(path "/b041be17-3693-4432-854e-c071e14fa049/af850077-64b1-47dc-8b85-ef279fd6955a"
-					(reference "V8")
+					(reference "V87")
 					(unit 1)
 				)
@@
 					(page "17")
 				)
-				(path "/b041be17-3693-4432-854e-c071e14fa049/af850077-64b1-47dc-8b85-ef279fd6955a"
-					(page "68")
-				)
 			)
