File: testbench_fa8_full.kicad_sch (KiCad schematic)
At the start: 0 parts

Commit message: FA8 full sim, before FA1 layout
Parts:
- added V_FA8_Test_A1, V_FA8_Test_A10, V_FA8_Test_A11, V_FA8_Test_A12, V_FA8_Test_A13, V_FA8_Test_A14, V_FA8_Test_A15, V_FA8_Test_A16, V_FA8_Test_A2, V_FA8_Test_A3, V_FA8_Test_A4, V_FA8_Test_A5, V_FA8_Test_A6, V_FA8_Test_A7, V_FA8_Test_A8, V_FA8_Test_A9: 5, symbol Simulation_SPICE:VDC
Connections:
- net GND: now also V_FA8_Test_A1.2, V_FA8_Test_A10.2, V_FA8_Test_A11.2, V_FA8_Test_A12.2, V_FA8_Test_A13.2, V_FA8_Test_A14.2, V_FA8_Test_A15.2, V_FA8_Test_A16.2, V_FA8_Test_A2.2, V_FA8_Test_A3.2, V_FA8_Test_A4.2, V_FA8_Test_A5.2, V_FA8_Test_A6.2, V_FA8_Test_A7.2, V_FA8_Test_A8.2, V_FA8_Test_A9.2
- new net IN_A0: V_FA8_Test_A1.1
- new net IN_A1: V_FA8_Test_A2.1
- new net IN_A2: V_FA8_Test_A3.1
- new net IN_A3: V_FA8_Test_A4.1
- new net IN_A4: V_FA8_Test_A5.1
- new net IN_A5: V_FA8_Test_A6.1
- new net IN_A6: V_FA8_Test_A7.1
- new net IN_A7: V_FA8_Test_A8.1
- new net IN_B0: V_FA8_Test_A9.1
- new net IN_B1: V_FA8_Test_A10.1
- new net IN_B2: V_FA8_Test_A11.1
- new net IN_B3: V_FA8_Test_A12.1
- new net IN_B4: V_FA8_Test_A13.1
- new net IN_B5: V_FA8_Test_A14.1
- new net IN_B6: V_FA8_Test_A15.1
- new net IN_B7: V_FA8_Test_A16.1
Other:
- note added: ".control define getbit8(num, pos) (num / (2 ^ pos)) % 2 echo Start Simulating FA 8-Bit let i = 0 let range_a = 256 let fail_count = 0 while i < range_a let vala = $&i let ran_cin = rnd(2) * 5 let j = 1 while j < 9 let jj = $&j - 1 set jj=$&jj let x = getbit8($&vala, $&jj) * 5 set j=$&j set Vname=V_FA8_Test_A{$j} alter $Vname $&x let j = j + 1 end ;echo vala = $&vala binary = $&x ; repeat 1 let va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"
- note added: "Tutorial: ngspice control language"
