File: testbench_gates.kicad_sch (KiCad schematic)
At the start: 2 parts

Commit message: FA 2-bit
Parts:
- renumbered V2 to V82, V3 to V83
Changed lines of the file:
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@@
 		(dnp no)
 		(fields_autoplaced yes)
-		(property "Reference" "V2"
+		(property "Reference" "V82"
 			(at 124.46 128.1401 0)
 			(effects
@@
 			(project "ICD24_FA"
 				(path "/b041be17-3693-4432-854e-c071e14fa049/bf61237c-4d83-41f1-a6ca-83160467bc81"
-					(reference "V2")
+					(reference "V82")
 					(unit 1)
 				)
@@
 		(dnp no)
 		(fields_autoplaced yes)
-		(property "Reference" "#PWR03"
+		(property "Reference" "#PWR083"
 			(at 120.65 144.78 0)
 			(effects
@@
 			(project "ICD24_FA"
 				(path "/b041be17-3693-4432-854e-c071e14fa049/bf61237c-4d83-41f1-a6ca-83160467bc81"
-					(reference "#PWR03")
+					(reference "#PWR083")
 					(unit 1)
 				)
@@
 		(dnp no)
 		(fields_autoplaced yes)
-		(property "Reference" "#PWR04"
+		(property "Reference" "#PWR084"
 			(at 120.65 168.91 0)
 			(effects
@@
 			(project "ICD24_FA"
 				(path "/b041be17-3693-4432-854e-c071e14fa049/bf61237c-4d83-41f1-a6ca-83160467bc81"
-					(reference "#PWR04")
+					(reference "#PWR084")
 					(unit 1)
 				)
@@
 		(dnp no)
 		(fields_autoplaced yes)
-		(property "Reference" "V3"
+		(property "Reference" "V83"
 			(at 124.46 153.5401 0)
 			(effects
@@
 			(project "ICD24_FA"
 				(path "/b041be17-3693-4432-854e-c071e14fa049/bf61237c-4d83-41f1-a6ca-83160467bc81"
-					(reference "V3")
+					(reference "V83")
 					(unit 1)
 				)
