File: xnor_gate.kicad_sch (KiCad schematic)
At the start: 11 parts, among them Q15 2N3904, Q16 2N3904, Q17 2N3904, Q18 2N3904

Commit message: full, no layout
Parts:
- removed Q15, Q16, Q17, Q18: 2N3904, Package_TO_SOT_THT:TO-92_Inline, symbol Transistor_BJT:2N3904
- added Q10, Q11, Q12, Q13: 2N3904, Package_TO_SOT_THT:TO-92_Inline, symbol Transistor_BJT:2N3904
- renumbered R22 to R14, R23 to R15, R24 to R16, R25 to R17, R26 to R18, R27 to R19, R28 to R20
Connections:
- net GND: now also Q11.1 (E), Q13.1 (E)
- net OUT: now also Q10.3 (C), Q12.3 (C)
- net at R15.2: now also Q13.2 (B)
- net at R18.2, R19.1: now also Q12.1 (E), Q13.3 (C)
- net at R16.1: now also Q12.2 (B)
- net at R18.1: now also Q10.2 (B)
- net at R16.2, R17.1: now also Q10.1 (E), Q11.3 (C)
- net at R14.2: now also Q11.2 (B)

Commit message: FA 2-bit
Parts:
- renumbered Q12 to Q90, Q10 to Q91, Q13 to Q92, Q11 to Q93, R14 to R100, R20 to R94, R18 to R95, R19 to R96, R16 to R97, R17 to R98, R15 to R99
Changed lines of the file:
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@@
 		(dnp no)
 		(fields_autoplaced yes)
-		(property "Reference" "R15"
+		(property "Reference" "R99"
 			(at 74.9299 113.03 0)
 			(effects
@@
 			(project "ICD24_FA"
 				(path "/b041be17-3693-4432-854e-c071e14fa049/bf61237c-4d83-41f1-a6ca-83160467bc81/c163f0a8-7b19-4740-9c97-b60a1695cc8f"
-					(reference "R15")
+					(reference "R99")
 					(unit 1)
 				)
@@
 		(dnp no)
 		(fields_autoplaced yes)
-		(property "Reference" "R20"
+		(property "Reference" "R94"
 			(at 187.96 57.1499 0)
 			(effects
@@
 			(project "ICD24_FA"
 				(path "/b041be17-3693-4432-854e-c071e14fa049/bf61237c-4d83-41f1-a6ca-83160467bc81/c163f0a8-7b19-4740-9c97-b60a1695cc8f"
-					(reference "R20")
+					(reference "R94")
 					(unit 1)
 				)
@@
 		(dnp no)
 		(fields_autoplaced yes)
-		(property "Reference" "R18"
+		(property "Reference" "R95"
 			(at 119.3799 85.09 0)
 			(effects
@@
 			(project "ICD24_FA"
 				(path "/b041be17-3693-4432-854e-c071e14fa049/bf61237c-4d83-41f1-a6ca-83160467bc81/c163f0a8-7b19-4740-9c97-b60a1695cc8f"
-					(reference "R18")
+					(reference "R95")
 					(unit 1)
 				)
@@
 		(dnp no)
 		(fields_autoplaced yes)
-		(property "Reference" "Q12"
+		(property "Reference" "Q90"
 			(at 132.08 76.1999 0)
 			(effects
@@
 			(project "ICD24_FA"
 				(path "/b041be17-3693-4432-854e-c071e14fa049/bf61237c-4d83-41f1-a6ca-83160467bc81/c163f0a8-7b19-4740-9c97-b60a1695cc8f"
-					(reference "Q12")
+					(reference "Q90")
 					(unit 1)
 				)
@@
 		(dnp no)
 		(fields_autoplaced yes)
-		(property "Reference" "R17"
+		(property "Reference" "R98"
 			(at 95.2499 102.87 0)
 			(effects
@@
 			(project "ICD24_FA"
 				(path "/b041be17-3693-4432-854e-c071e14fa049/bf61237c-4d83-41f1-a6ca-83160467bc81/c163f0a8-7b19-4740-9c97-b60a1695cc8f"
-					(reference "R17")
+					(reference "R98")
 					(unit 1)
 				)
@@
 		(dnp no)
 		(fields_autoplaced yes)
-		(property "Reference" "Q10"
+		(property "Reference" "Q91"
 			(at 90.17 93.9799 0)
 			(effects
@@
 			(project "ICD24_FA"
 				(path "/b041be17-3693-4432-854e-c071e14fa049/bf61237c-4d83-41f1-a6ca-83160467bc81/c163f0a8-7b19-4740-9c97-b60a1695cc8f"
-					(reference "Q10")
+					(reference "Q91")
 					(unit 1)
 				)
@@
 		(dnp no)
 		(fields_autoplaced yes)
-		(property "Reference" "R19"
+		(property "Reference" "R96"
 			(at 138.4299 85.09 0)
 			(effects
@@
 			(project "ICD24_FA"
 				(path "/b041be17-3693-4432-854e-c071e14fa049/bf61237c-4d83-41f1-a6ca-83160467bc81/c163f0a8-7b19-4740-9c97-b60a1695cc8f"
-					(reference "R19")
+					(reference "R96")
 					(unit 1)
 				)
@@
 		(dnp no)
 		(fields_autoplaced yes)
-		(property "Reference" "Q13"
+		(property "Reference" "Q92"
 			(at 132.08 114.2999 0)
 			(effects
@@
 			(project "ICD24_FA"
 				(path "/b041be17-3693-4432-854e-c071e14fa049/bf61237c-4d83-41f1-a6ca-83160467bc81/c163f0a8-7b19-4740-9c97-b60a1695cc8f"
-					(reference "Q13")
+					(reference "Q92")
 					(unit 1)
 				)
@@
 		(dnp no)
 		(fields_autoplaced yes)
-		(property "Reference" "R16"
+		(property "Reference" "R97"
 			(at 76.1999 102.87 0)
 			(effects
@@
 			(project "ICD24_FA"
 				(path "/b041be17-3693-4432-854e-c071e14fa049/bf61237c-4d83-41f1-a6ca-83160467bc81/c163f0a8-7b19-4740-9c97-b60a1695cc8f"
-					(reference "R16")
+					(reference "R97")
 					(unit 1)
 				)
@@
 		(dnp no)
 		(fields_autoplaced yes)
-		(property "Reference" "Q11"
+		(property "Reference" "Q93"
 			(at 90.17 125.7299 0)
 			(effects
@@
 			(project "ICD24_FA"
 				(path "/b041be17-3693-4432-854e-c071e14fa049/bf61237c-4d83-41f1-a6ca-83160467bc81/c163f0a8-7b19-4740-9c97-b60a1695cc8f"
-					(reference "Q11")
+					(reference "Q93")
 					(unit 1)
 				)
@@
 		(dnp no)
 		(fields_autoplaced yes)
-		(property "Reference" "R14"
+		(property "Reference" "R100"
 			(at 72.3899 124.46 0)
 			(effects
@@
 			(project "ICD24_FA"
 				(path "/b041be17-3693-4432-854e-c071e14fa049/bf61237c-4d83-41f1-a6ca-83160467bc81/c163f0a8-7b19-4740-9c97-b60a1695cc8f"
-					(reference "R14")
-					(unit 1)
-				)
+					(reference "R100")
+					(unit 1)
+				)
